File: hardware/pcb/binfohub_bridge.kicad_pcb (KiCad board)
At the start: 2 copper layers, 90 x 92 mm, 48 parts, among them J1 12V IN, J2 BUS A B, J3 IH 12V GND A B, J4 LED OUT, Q1 AO3401A, U1 ESP32-DevKitC-32 (38-pin), U2 AP63205WU-7, U3 SP3485EN, U4 SP3485EN

Commit message: Hardware rev 1.1: bare WROOM-32E, 3.3 V rail, fan header, programming header
Same outline, holes, terminal and LED positions as rev 1.0, so it fits the
existing enclosure. Driven by the 2026-10-01 thermal failure: ESP32-WROOM-32E
soldered at the right edge (antenna outward; -32UE fits the same pads for a
U.FL remote antenna), AP63203 3.3 V buck replacing the 5 V rail and the
DevKit's linear regulator, J5 12 V PWM fan output (IO32, AO3400A, F3, SS14),
EN/IO0 support with RESET/BOOT and a J6 programming header, R10/R11 bias.

ERC 0, DRC 0 errors / 0 unconnected (7 cosmetic warnings), 100 % routed
(755 tracks / 104 vias), ground pour plotted. Rev 1.0's shipped gerbers had
no pour (zone outlines were never refilled at plot time); export.sh now
refills and counts regions. Router gains a --trim-only mode and a junction-
aware dangling-end trim. packages/fan.yaml added (commented include; RAM
83.0 %, see its header). Rev 1.0 files tagged pcb-rev1.0.

Co-Authored-By: Claude Fable 5.1 <noreply@anthropic.com>
Claude-Session: https://claude.ai/code/session_01ESVh7DpLzA3jfcrFtGgM8a
Parts:
- added C11: 1uF 50V, Capacitor_SMD:C_0603_1608Metric, F.Cu at (61.0, 49.0)
- added D10: SS14, Diode_SMD:D_SMA, F.Cu at (37.5, 47.5)
- added F3: 0.5A polyfuse 1812, Fuse:Fuse_1812_4532Metric, F.Cu at (37.5, 42.0)
- added J5: FAN 12V, TerminalBlock_Phoenix:TerminalBlock_Phoenix_MPT-0,5-2-2.54_1x02_P2.54mm_Horizontal, F.Cu at (30.5, 42.0)
- added J6: PROG, Connector_PinHeader_2.54mm:PinHeader_1x06_P2.54mm_Vertical, F.Cu at (14.0, 50.0)
- added Q2: AO3400A, Package_TO_SOT_SMD:SOT-23, F.Cu at (29.0, 51.0)
- added R10: 4k7, Resistor_SMD:R_0603_1608Metric, F.Cu at (66.0, 25.0)
- added R11: 4k7, Resistor_SMD:R_0603_1608Metric, F.Cu at (66.0, 29.0)
- added R12: 100R, Resistor_SMD:R_0603_1608Metric, F.Cu at (23.0, 51.0)
- added R13: 10k, Resistor_SMD:R_0603_1608Metric, F.Cu at (23.0, 55.0)
- added R14: 10k, Resistor_SMD:R_0603_1608Metric, F.Cu at (65.0, 49.0)
- added R15: 10k, Resistor_SMD:R_0603_1608Metric, F.Cu at (47.0, 71.5)
- added SW1: TS-1187A, binfohub:SW_TS-1187A, F.Cu at (57.0, 42.0)
- added SW2: TS-1187A, binfohub:SW_TS-1187A, F.Cu at (69.0, 42.0)
- C7: value 22uF 25V -> 10uF 25V
- R5: value 330R -> 100R
- U1: value ESP32-DevKitC-32 (38-pin) -> ESP32-WROOM-32E; footprint binfohub:ESP32-DevKitC-38 -> binfohub:ESP32-WROOM-32E_edge
- U2: value AP63205WU-7 -> AP63203WU-7
- moved J4 77.0 mm to (8.00, 54.0)
- moved C8 35.6 mm to (72.5, 46.5), turned to 0 degrees
- moved C7 33.6 mm to (69.0, 49.0), turned to 0 degrees
- moved U1 22.1 mm to (66.0, 62.0), turned to 270 degrees
- moved C10 14.0 mm to (64.5, 33.0)
- moved R5 2.50 mm to (18.0, 77.5)
- moved R6 2.50 mm to (29.0, 77.5)
- moved R7 2.50 mm to (40.0, 77.5)
- moved R8 2.50 mm to (51.0, 77.5)
- moved R9 2.50 mm to (62.0, 77.5)
- moved F2 0.50 mm to (45.5, 33.5)
Connections:
- net 5V_BUCK renamed 3V3_BUCK
- C7 pad 1: +5V -> +3V3
- C8 pad 1: +5V -> +3V3
- F1 pad 2: +5V -> +3V3
- R5 pad 1: +5V -> +3V3
- U1 pad 1: +3V3 -> GND
- U1 pad 10: LED_BUS -> LED_WIFI
- U1 pad 11: LED_FAULT -> LED_BUS
- U1 pad 12: unconnected-(U1-IO14-Pad12) -> LED_FAULT
- U1 pad 14: GND -> unconnected-(U1-IO12-Pad14)
- U1 pad 15: unconnected-(U1-IO13-Pad15) -> GND
- U1 pad 19: +5V -> unconnected-(U1-NC-Pad19)
- U1 pad 2: unconnected-(U1-EN-Pad2) -> +3V3
- U1 pad 20: GND -> unconnected-(U1-NC-Pad20)
- U1 pad 21: B_RO -> unconnected-(U1-NC-Pad21)
- U1 pad 22: B_DI -> unconnected-(U1-NC-Pad22)
- U1 pad 25: B_DE -> ESP_IO0
- U1 pad 26: GND -> A_DE
- U1 pad 27: unconnected-(U1-IO19-Pad27) -> A_RO
- U1 pad 28: unconnected-(U1-IO18-Pad28) -> A_DI
- U1 pad 3: unconnected-(U1-IO36/VP-Pad3) -> ESP_EN
- U1 pad 30: A_DI -> unconnected-(U1-IO18-Pad30)
- U1 pad 31: A_RO -> unconnected-(U1-IO19-Pad31)
- U1 pad 32: A_DE -> unconnected-(U1-NC-Pad32)
- U1 pad 33: unconnected-(U1-IO0-Pad33) -> B_DE
- U1 pad 34: unconnected-(U1-IO2-Pad34) -> ESP_RXD0
- U1 pad 35: unconnected-(U1-IO15-Pad35) -> ESP_TXD0
- U1 pad 36: unconnected-(U1-IO8/SD1-Pad36) -> B_DI
- U1 pad 37: unconnected-(U1-IO7/SD0-Pad37) -> B_RO
- U1 pad 38: unconnected-(U1-IO6/CLK-Pad38) -> GND
- U1 pad 8: unconnected-(U1-IO33-Pad8) -> FAN_PWM
- U1 pad 9: LED_WIFI -> unconnected-(U1-IO33-Pad9)
Routing:
- net +5V: track 127.3 -> 0.00 mm, vias 5 -> 0
- net LED_WIFI: track 16.6 -> 104.4 mm, vias 1 -> 4
- net ESP_TXD0: track 0.00 -> 85.7 mm, vias 0 -> 7
- net ESP_IO0: track 0.00 -> 83.3 mm, vias 0 -> 4
- net ESP_EN: track 0.00 -> 77.6 mm, vias 0 -> 2
- net ESP_RXD0: track 0.00 -> 70.5 mm, vias 0 -> 4
- net FAN_PWM: track 0.00 -> 64.1 mm, vias 0 -> 4
- net GND: track 275.7 -> 329.2 mm, vias 4 -> 11
- net +3V3: track 133.5 -> 184.6 mm, vias 4 -> 5
- net A_DI: track 32.1 -> 83.0 mm, vias 2 -> 4
- net LED_PWR: track 77.5 -> 29.6 mm
- net B_DE: track 45.0 -> 89.0 mm, vias 2 -> 4
- net LED_TX_A: track 29.2 -> 70.1 mm, vias 0 -> 2
- net IH_B: track 34.0 -> 73.2 mm, vias 2 -> 7
- net LED_WIFI_A: track 70.4 -> 33.8 mm, vias 1 -> 3
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Other:
- board text added: "2026-10 bbensten"
- board text added: "3V3"
- board text added: "ANT >"
- board text added: "B-INFOHUB BRIDGE v1.1"
- board text added: "BOOT"
- board text added: "EN"
- board text added: "ESP32-WROOM-32E. Fit -32UE + U.FL pigtail for a remote antenna."
- board text added: "F1 1.1A feeds the bridge, F2 2A the InfoHub, F3 0.5A the fan - separate"
- board text added: "IO0"
- board text added: "J5 FAN"
- board text added: "J5 FAN 12V 0.5A PWM (IO32). J6 PROG: first flash only, then OTA."
- board text added: "J6 PROG"
- board text added: "RESET"
- board text added: "RX"
- board text added: "SW"
- board text added: "on purpose: no single fault takes the telemetry down."
- board text removed: "2026-08 bbensten"
- board text removed: "B-INFOHUB BRIDGE v1.0"
- board text removed: "ESP32-DevKitC-32, or -32U if you need an external antenna"
- board text removed: "F1 1.1A feeds the bridge, F2 2A feeds the InfoHub - separate on purpose:"
- board text removed: "the InfoHub cell modem pulses hard and must not take the telemetry down."

Commit message: PCB rev 1.1: EE review fixes
-H4 (105 C) module C3013935; DE pull-downs R16/R17 so neither transceiver can
drive the bus while the ESP is in reset or being flashed; 680R fail-safe bias
(covers a terminated far end); F3 1.1 A / 33 V (a 0.5 A PPTC derates below
any real fan at box temperature); 100 nF at the VDD pad; BOM grouped by part
so no LCSC number spans two lines; header rotation keys fixed; JLC gerber set
trimmed to fab layers. ERC 0, DRC 0 errors / 0 unconnected, 738 tracks / 109
vias, pour plotted.

Co-Authored-By: Claude Fable 5.1 <noreply@anthropic.com>
Claude-Session: https://claude.ai/code/session_01ESVh7DpLzA3jfcrFtGgM8a
Parts:
- added R16: 10k, Resistor_SMD:R_0603_1608Metric, F.Cu at (46.0, 30.5)
- added R17: 10k, Resistor_SMD:R_0603_1608Metric, F.Cu at (61.0, 29.0)
- F3: value 0.5A polyfuse 1812 -> 1.1A polyfuse 1812 33V
- R10, R11: value 4k7 -> 680R
- U1: value ESP32-WROOM-32E -> ESP32-WROOM-32E-H4
- moved C7 4.30 mm to (72.5, 46.5)
- moved C8 4.30 mm to (69.0, 49.0)
Routing:
- net B_DI: track 43.0 -> 200.1 mm, vias 2 -> 6
- net LED_WIFI: track 104.4 -> 47.1 mm, vias 4 -> 0
- net ESP_IO0: track 83.3 -> 139.2 mm, vias 4 -> 6
- net GND: track 329.2 -> 360.8 mm, vias 11 -> 9
- net B_DE: track 89.0 -> 58.1 mm, vias 4 -> 2
- net IH_B: track 73.2 -> 55.5 mm, vias 7 -> 3
- net ESP_TXD0: track 85.7 -> 96.8 mm, vias 7 -> 1
- net BUS_A: track 36.9 -> 47.2 mm, vias 3 -> 4
- net A_DI: track 83.0 -> 73.0 mm, vias 4 -> 6
- net FAN_PWM: track 64.1 -> 54.7 mm, vias 4 -> 6
- net A_RO: track 85.9 -> 77.7 mm
- net ESP_RXD0: track 70.5 -> 64.3 mm, vias 4 -> 6
- net ESP_EN: track 77.6 -> 73.1 mm, vias 2 -> 4
- net LED_FLT_A: track 59.0 -> 54.7 mm, vias 4 -> 2
- net LED_BUS: track 35.6 -> 31.5 mm, vias 0 -> 2
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Other:
- board text added: "F1 1.1A feeds the bridge, F2 2A the InfoHub, F3 1.1A the fan - separate"
- board text added: "J5 FAN 12V <=0.5A PWM (IO32). J6 PROG: first flash only, then OTA."
- board text removed: "F1 1.1A feeds the bridge, F2 2A the InfoHub, F3 0.5A the fan - separate"
- board text removed: "J5 FAN 12V 0.5A PWM (IO32). J6 PROG: first flash only, then OTA."
